File: TDA2005R/TDA2005R-1.0.kicad_pcb (KiCad board)
At the start: 2 copper layers, 71.8 x 85.1 mm, 30 parts, among them J1 6-pole_dual_potentiometer_hea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, U1 4-pole_RL-input_screw_terminal, U2 TDA2005, U3 4-pole_RL-output_screw_termin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, U4 2-pole_power_in_screw_terminal

Commit message: kicad6
Other:
- net class 30 removed
- net class 50 removed
- net class Default removed
