File: TDA2005R/TDA2005R-1.1.kicad_sch (KiCad schematic)
At the start: 26 parts

Commit message: amplifier
Parts:
- removed C1, C10, C11, C2, C3, C4, C5, C6, C7: (no value), symbol Device:CP
- removed J1: (no value), symbol My_Headers:6-pole_dual_potentiometer_header
- removed RV1: (no value), symbol Device:R_POT_Dual
- removed U1: (no value), symbol My_Parts:4-pole_RL-input_screw_terminal
- added C1, C2: 2.2u, My_Misc:CP_Radial_D5.0mm_P2.00mm_larger, symbol Device:C_Polarized
- added C10, C11: 2200u, My_Misc:CP_Radial_D13.0mm_P5.00mm_larger, symbol Device:C_Polarized
- added C3: 10u, My_Misc:CP_Radial_D5.0mm_P2.00mm_larger, symbol Device:C_Polarized
- added C4, C6: 100u, My_Misc:CP_Radial_D5.0mm_P2.50mm_larger_pads, symbol Device:C_Polarized
- added C5, C7: 220u, My_Misc:CP_Radial_D8.0mm_P3.50mm_large, symbol Device:C_Polarized
- added H1, H2, H3, H4: MountingHole, MountingHole:MountingHole_3.2mm_M3, symbol Mechanical:MountingHole
- added J1: Audio In, My_Headers:3-pin JST Audio, symbol My_Headers:3-pin_Audio
- added U1: Vol R, My_Headers:3-pin JST Potentiometer, symbol My_Headers:3-pin_potentiometer_output
- added U2: Vol L, My_Headers:3-pin JST Potentiometer, symbol My_Headers:3-pin_potentiometer_output
- C12: value (none) -> 0.1u; footprint (none) -> My_Misc:C_Disc_D7.5mm_W2.5mm_P5.00mm_larger
- C8: renamed from C9; value (none) -> 0.1u; footprint (none) -> My_Misc:C_Disc_D7.5mm_W2.5mm_P5.00mm_larger
- C9: renamed from C8; value (none) -> 0.1u; footprint (none) -> My_Misc:C_Disc_D7.5mm_W2.5mm_P5.00mm_larger
- HS1: value (none) -> Heatsink_Pad; footprint (none) -> My_Heatsinks:EK-41002859
- R1: value (none) -> 120k; footprint (none) -> My_Misc:R_Axial_DIN0414_L11.9mm_D4.5mm_P15.24mm_Horizontal_larger
- R2: renamed from R4; value (none) -> 1.2k; footprint (none) -> My_Misc:R_Axial_DIN0414_L11.9mm_D4.5mm_P15.24mm_Horizontal_larger
- R3: renamed from R5; value (none) -> 3R3; footprint (none) -> My_Misc:R_Axial_DIN0414_L11.9mm_D4.5mm_P15.24mm_Horizontal_larger
- R4: renamed from R2; value (none) -> 1.2k; footprint (none) -> My_Misc:R_Axial_DIN0414_L11.9mm_D4.5mm_P15.24mm_Horizontal_larger
- R5: renamed from R3; value (none) -> 3R3; footprint (none) -> My_Misc:R_Axial_DIN0414_L11.9mm_D4.5mm_P15.24mm_Horizontal_larger
- R6: renamed from R7; value (none) -> 1R; footprint (none) -> My_Misc:R_Axial_DIN0414_L11.9mm_D4.5mm_P15.24mm_Horizontal_larger
- R7: renamed from R6; value (none) -> 1R; footprint (none) -> My_Misc:R_Axial_DIN0414_L11.9mm_D4.5mm_P15.24mm_Horizontal_larger
- U3: renamed from U2; value (none) -> TDA2005; footprint (none) -> My_Misc:TO-220-11_P3.4x5.08mm_StaggerOdd_Lead4.85mm_Vertical_large
- U4: renamed from U3; value (none) -> Speakers; footprint (none) -> My_Parts:4-pole_screw_terminal_RL_output
- U5: renamed from U4; value (none) -> Power In; footprint (none) -> My_Parts:2-pole_power_in_screw_terminal
Connections:
- net GND: now also C3.2, J1.3 (-), U1.3 (PB0), U2.3 (PB0)
- net Lin: now also J1.2 (L+), U2.1 (PAO)
- net Lout: now also C10.1
- net Rin: now also J1.1 (R+), U1.1 (PAO)
- net Rout: now also C11.1
- net at U3.1 (+): now also C2.1
- net at C9.1, R4.1, U3.10: now also C11.2, C6.2
- net at U3.11 (BOOT): now also C6.1
- net at U3.2 (-): now also C7.1
- net at R1.2, U3.3 (SVRR): now also C3.1
- net at U3.4 (-): now also C5.1
- net at U3.5 (+): now also C1.1
- net at U3.7 (BOOT): now also C4.1
- net at C8.1, R2.1, U3.8: now also C10.2, C4.2
- net at R4.2, R5.1: now also C7.2
- net at R2.2, R3.1: now also C5.2
- new net: C1.2, U2.2 (PW0)
- new net: C2.2, U1.2 (PW0)
