File: TDA2005-amplifiers/1-channel_bridged_amplifier.kicad_sch (KiCad schematic)
At the start: 19 parts

Commit message: bridged amplifier
Parts:
- removed C1, C2, C4, C5, C6, C7, C8: (no value), symbol Device:CP
- added C1, C2: 2.2u/3V, My_Misc:CP_Radial_D5.0mm_P2.00mm_larger, symbol Device:C_Polarized
- added C4: 10u, My_Misc:CP_Radial_D5.0mm_P2.00mm_larger, symbol Device:C_Polarized
- added C5, C7: 100u/10V, My_Misc:CP_Radial_D8.0mm_P3.50mm_large, symbol Device:C_Polarized
- added C6, C8: 220u/3V, My_Misc:CP_Radial_D10.0mm_P5.00mm_larger, symbol Device:C_Polarized
- added H1, H3, H4: MountingHole, MountingHole:MountingHole_3.2mm_M3, symbol Mechanical:MountingHole
- added HS1: Heatsink_Pad, My_Heatsinks:EK-41002859, symbol Mechanical:Heatsink_Pad
- added J1: Audio In, My_Headers:2-pin JST Audio, symbol My_Headers:2-pin_Audio
- added U2: Speaker Out, My_Parts:2-pole_power_in_screw_terminal, symbol My_Parts:2-pole_power_in_screw_terminal
- C10, C3, C9: value (none) -> 100n; footprint (none) -> My_Misc:C_Disc_D7.5mm_W2.5mm_P5.00mm_larger
- R1: value (none) -> 120k; footprint (none) -> My_Misc:R_Axial_DIN0414_L11.9mm_D4.5mm_P15.24mm_Horizontal_larger
- R2, R3A1, R3B1: value (none) -> 1k; footprint (none) -> My_Misc:R_Axial_DIN0414_L11.9mm_D4.5mm_P15.24mm_Horizontal_larger
- R4, R5: value (none) -> 12R; footprint (none) -> My_Misc:R_Axial_DIN0414_L11.9mm_D4.5mm_P15.24mm_Horizontal_larger
- R6, R7: value (none) -> 1R; footprint (none) -> My_Misc:R_Axial_DIN0414_L11.9mm_D4.5mm_P15.24mm_Horizontal_larger
- U1: value (none) -> TDA2005; footprint (none) -> My_Misc:TO-220-11_P3.4x5.08mm_StaggerOdd_Lead4.85mm_Vertical_large
Connections:
- net GND: now also C2.2, C4.2, HS1.1, J1.2 (-)
- net at U1.1 (+): now also C1.1
- net at U1.11 (BOOT): now also C5.1
- net at U1.2 (-): now also C6.1
- net at R1.2, U1.3 (SVRR): now also C4.1
- net at U1.4 (-): now also C8.1
- net at U1.5 (+): now also C2.1
- net at U1.7 (BOOT): now also C7.1
- net at R2.2, R4.1, R5.1: now also C6.2
- net at R3B1.2, R4.2: now also C8.2
- net Out+: no longer names the net of C9.1, R2.1, U1.10
- net Out+: now also C5.2, U2.1 (+)
- net Out-: no longer names the net of C10.1, R3A1.1, U1.8
- net Out-: now also C7.2, U2.2 (-)
- new net: C1.2, J1.1 (+)
Other:
- moved on the sheet: C3, U1C
