File: TDA2005-amplifiers/2-channel_tone,_balance_and_loudness_amplifier.kicad_sch (KiCad schematic)
At the start: 41 parts

Commit message: 2-channel
Parts:
- removed C12, C13, C14, C15, C16, C19, C20: (no value), symbol Device:CP
- removed RV1: (no value), symbol Device:R_POT
- removed U2: (no value), symbol My_Parts:4-pole_RL-input_screw_terminal
- added C?: 10u, symbol Device:C_Polarized
- added C? (x4): 100u, symbol Device:C_Polarized
- added C? (x2): 2200u, symbol Device:C_Polarized
- added J?: 3-pin_Audio, symbol My_Headers:3-pin_Audio
- added RV?: 100k, symbol Device:R_Potentiometer
- C1, C2: value (none) -> 47n; footprint (none) -> My_Misc:C_Disc_D7.5mm_W2.5mm_P5.00mm_larger
- C10, C11: value (none) -> 220n; footprint (none) -> My_Misc:C_Disc_D7.5mm_W2.5mm_P5.00mm_larger
- C17, C18, C7: value (none) -> 100n; footprint (none) -> My_Misc:C_Disc_D7.5mm_W2.5mm_P5.00mm_larger
- C3, C5, C8, C9: value (none) -> 2.2n; footprint (none) -> My_Misc:C_Disc_D7.5mm_W2.5mm_P5.00mm_larger
- C4, C6: value (none) -> 150n; footprint (none) -> My_Misc:C_Disc_D7.5mm_W2.5mm_P5.00mm_larger
- HS1: value (none) -> Heatsink_Pad; footprint (none) -> My_Heatsinks:EK-41002859
- R1, R2: value (none) -> 5.6k; footprint (none) -> My_Misc:R_Axial_DIN0414_L11.9mm_D4.5mm_P15.24mm_Horizontal_larger
- R10, R8: value (none) -> 100k; footprint (none) -> My_Misc:R_Axial_DIN0414_L11.9mm_D4.5mm_P15.24mm_Horizontal_larger
- R11, R9: value (none) -> 3.3R; footprint (none) -> My_Misc:R_Axial_DIN0414_L11.9mm_D4.5mm_P15.24mm_Horizontal_larger
- R12, R13: value (none) -> 1R; footprint (none) -> My_Misc:R_Axial_DIN0414_L11.9mm_D4.5mm_P15.24mm_Horizontal_larger
- R3, R5: value (none) -> 47k; footprint (none) -> My_Misc:R_Axial_DIN0414_L11.9mm_D4.5mm_P15.24mm_Horizontal_larger
- R4, R6: value (none) -> 2.7k; footprint (none) -> My_Misc:R_Axial_DIN0414_L11.9mm_D4.5mm_P15.24mm_Horizontal_larger
- R7: value (none) -> 120k; footprint (none) -> My_Misc:R_Axial_DIN0414_L11.9mm_D4.5mm_P15.24mm_Horizontal_larger
- RV1-1, RV3-1: value (none) -> Dual_potentiometer; footprint (none) -> My_Misc:Potentiometer_Piher_PC-16_Dual_Horizontal_larger
- U1: value (none) -> TDA2005; footprint (none) -> My_Misc:TO-220-11_P3.4x5.08mm_StaggerOdd_Lead4.85mm_Vertical_large
- U3: value (none) -> 2-pole_power_in_screw_terminal; footprint (none) -> My_Parts:2-pole_power_in_screw_terminal
- U4: value (none) -> 4-pole_RL-output_screw_terminal; footprint (none) -> My_Parts:4-pole_screw_terminal_RL_output
Connections:
- net GND: now also C?.2, J?.3 (-), RV?.2
- net Lin+: now also J?.2 (L+)
- net Lout+: now also C?.2
- net Rin+: now also J?.1 (R+)
- net Rout+: now also C?.2
- net at C17.1, R8.1, U1.10: now also C?.1, C?.2
- net at U1.11 (BOOT): now also C?.1
- net at U1.2 (-): now also C?.1
- net at R7.2, U1.3 (SVRR): now also C?.1
- net at U1.4 (-): now also C?.1
- net at U1.7 (BOOT): now also C?.1
- net at C18.1, R10.1, U1.8: now also C?.1, C?.2
- net at R8.2, R9.1: now also C?.2
- net at R10.2, R11.1: now also C?.2
- net at C10.2, C8.2, RV3-1.1 (2): now also RV?.1
- net at C11.2, C9.2, RV3-1.4 (5): now also RV?.3
