File: LCD BackPack/KiCad/LCD BackPack.kicad_sch (KiCad schematic)
At the start: 5 parts

Commit message: lcd backpack
Parts:
- removed J2: (no value), symbol Connector:Conn_01x02_Male
- added JP1: Jumper_2_Open, My_Parts:Angled_Jumper_1x02_P2.54mm_large, symbol Jumper:Jumper_2_Open
- J1: value (none) -> 10-pin_header_LCD_interface; footprint (none) -> My_Headers:10-pin_LCD_header_larger_pads
- R1: value (none) -> 220R; footprint (none) -> My_Misc:R_Axial_DIN0207_L6.3mm_D2.5mm_P10.16mm_Horizontal_larger_pads
- RV1: renamed from RV?; value R_Potentiometer -> Contrast; footprint (none) -> My_Misc:Potentiometer_Bourns_3339P_Vertical_large
- U1: value (none) -> LCD_HD44780; footprint (none) -> My_Parts:LCD_HD44780_16x2_w_headers_no outlinelarge
Connections:
- net GND: now reaches J1.1 (VSS), U1.1 (VSS), U1.5 (R/W)
- net GND: now also RV1.3, JP1.1 (A); no longer RV1.1
- net at J1.10 (LED-), U1.16 (LED-): now also JP1.2 (B)
- net at J1.2 (VDD), R1.1, U1.2 (VDD): now also RV1.1; no longer RV1.3
Other:
- note added: "When 10-pin connection is used: * no resistor R1 * no jumper JP1"
- note added: "When 8-pin connection is used: * add resistor R1, 220R, to power backlight * short jumper JP1 for backlight ground"
- note removed: "When 10-pin connection is used: * no resistor R1 * no jumper J2"
- note removed: "When 8-pin connection is used: * add resistor R1, 220R, to power backlight * short jumper J2 for backlight ground"
- moved on the sheet: RV1
Changed lines of the file:
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@@
-    (stroke (width 0) (type default) (color 0 0 0 0))
-  )
-  (wire (pts (xy 147.32 137.16) (xy 105.41 137.16))
     (stroke (width 0) (type default) (color 0 0 0 0))
   )
@@
     (stroke (width 0) (type default) (color 0 0 0 0))
   )
-  (wire (pts (xy 105.41 137.16) (xy 105.41 82.55))
-    (stroke (width 0) (type default) (color 0 0 0 0))
-  )
   (wire (pts (xy 123.19 85.09) (xy 162.56 85.09))
     (stroke (width 0) (type default) (color 0 0 0 0))
@@
     (stroke (width 0) (type default) (color 0 0 0 0))
   )
+  (wire (pts (xy 105.41 143.51) (xy 132.08 143.51))
+    (stroke (width 0) (type default) (color 0 0 0 0))
+  )
   (wire (pts (xy 168.91 63.5) (xy 168.91 87.63))
     (stroke (width 0) (type default) (color 0 0 0 0))
@@
     (stroke (width 0) (type default) (color 0 0 0 0))
   )
-  (wire (pts (xy 168.91 137.16) (xy 168.91 120.65))
+  (wire (pts (xy 168.91 120.65) (xy 168.91 143.51))
     (stroke (width 0) (type default) (color 0 0 0 0))
   )
@@
     (stroke (width 0) (type default) (color 0 0 0 0))
   )
-  (wire (pts (xy 149.86 137.16) (xy 168.91 137.16))
-    (stroke (width 0) (type default) (color 0 0 0 0))
-  )
   (wire (pts (xy 153.67 69.85) (xy 162.56 69.85))
     (stroke (width 0) (type default) (color 0 0 0 0))
@@
     (stroke (width 0) (type default) (color 0 0 0 0))
   )
+  (wire (pts (xy 142.24 143.51) (xy 168.91 143.51))
+    (stroke (width 0) (type default) (color 0 0 0 0))
+  )
   (wire (pts (xy 137.16 82.55) (xy 172.72 82.55))
     (stroke (width 0) (type default) (color 0 0 0 0))
@@
     (stroke (width 0) (type default) (color 0 0 0 0))
   )
+  (wire (pts (xy 105.41 82.55) (xy 105.41 143.51))
+    (stroke (width 0) (type default) (color 0 0 0 0))
+  )
   (wire (pts (xy 179.07 82.55) (xy 172.72 82.55))
     (stroke (width 0) (type default) (color 0 0 0 0))
   )
-  (text "When 10-pin connection is used:\n* no resistor R1\n* no jumper J2"
+  (text "When 10-pin connection is used:\n* no resistor R1\n* no jumper JP1"
     (at 175.26 139.7 0)
     (effects (font (size 1.27 1.27)) (justify left bottom))
   )
-  (text "When 8-pin connection is used:\n* add resistor R1, 220R, to power backlight\n* short jumper J2 for backlight ground"
+  (text "When 8-pin connection is used:\n* add resistor R1, 220R, to power backlight\n* short jumper JP1 for backlight ground"
     (at 175.26 132.08 0)
+    (effects (font (size 1.27 1.27)) (justify left bottom))
+  )
+  (label "GND" (at 130.81 82.55 0)
     (effects (font (size 1.27 1.27)) (justify left bottom))
   )
@@
       (effects (font (size 1.27 1.27)) (justify left))
     )
-    (property "Value" "" (id 1) (at 192.4812 102.616 0)
-      (effects (font (size 1.27 1.27)) (justify left))
-    )
-    (property "Footprint" "" (id 2) (at 205.74 125.73 0)
+    (property "Value" "LCD_HD44780" (id 1) (at 192.4812 102.616 0)
+      (effects (font (size 1.27 1.27)) (justify left))
+    )
+    (property "Footprint" "My_Parts:LCD_HD44780_16x2_w_headers_no outlinelarge" (id 2) (at 205.74 125.73 0)
       (effects (font (size 1.27 1.27)) hide)
     )
@@
       (effects (font (size 1.27 1.27)) (justify left))
     )
-    (property "Value" "" (id 1) (at 149.733 129.032 0)
-      (effects (font (size 1.27 1.27)) (justify left))
-    )
-    (property "Footprint" "" (id 2) (at 148.59 132.588 90)
+    (property "Value" "220R" (id 1) (at 149.733 129.032 0)
+      (effects (font (size 1.27 1.27)) (justify left))
+    )
+    (property "Footprint" "My_Misc:R_Axial_DIN0207_L6.3mm_D2.5mm_P10.16mm_Horizontal_larger_pads" (id 2) (at 148.59 132.588 90)
       (effects (font (size 1.27 1.27)) hide)
     )
@@
     (in_bom yes) (on_board yes)
     (property "Reference" "J1" (id 0) (at 91.6432 56.5658 0))
-    (property "Value" "" (id 1) (at 91.44 57.15 0)
-      (effects (font (size 1.27 1.27)) hide)
-    )
-    (property "Footprint" "" (id 2) (at 93.98 59.69 0)
+    (property "Value" "10-pin_header_LCD_interface" (id 1) (at 91.44 57.15 0)
+      (effects (font (size 1.27 1.27)) hide)
+    )
+    (property "Footprint" "My_Headers:10-pin_LCD_header_larger_pads" (id 2) (at 93.98 59.69 0)
       (effects (font (size 1.27 1.27)) hide)
     )
@@
     (pin "9")
   )
-  (symbol (lib_id "Connector:Conn_01x02_Male") (at 147.32 142.24 90) (unit 1)
-    (in_bom yes) (on_board yes)
-    (property "Reference" "J2" (id 0) (at 146.2024 140.6652 90)
-      (effects (font (size 1.27 1.27)) (justify left))
-    )
-    (property "Value" "" (id 1) (at 146.2024 138.3538 90)
-      (effects (font (size 1.27 1.27)) (justify left) hide)
-    )
-    (property "Footprint" "" (id 2) (at 147.32 142.24 0)
-      (effects (font (size 1.27 1.27)) hide)
-    )
-    (property "Datasheet" "~" (id 3) (at 147.32 142.24 0)
-      (effects (font (size 1.27 1.27)) hide)
-    )
-    (pin "1")
-    (pin "2")
-  )
-  (symbol (lib_id "Device:R_Potentiometer") (at 149.86 69.85 90) (unit 1)
+  (symbol (lib_id "Device:R_Potentiometer") (at 149.86 69.85 270) (mirror x) (unit 1)
     (in_bom yes) (on_board yes) (fields_autoplaced)
-    (property "Reference" "RV?" (id 0) (at 149.86 72.8964 90))
-    (property "Value" "R_Potentiometer" (id 1) (at 149.86 75.4333 90))
-    (property "Footprint" "" (id 2) (at 149.86 69.85 0)
+    (property "Reference" "RV1" (id 0) (at 149.86 72.8964 90))
+    (property "Value" "Contrast" (id 1) (at 149.86 75.4333 90))
+    (property "Footprint" "My_Misc:Potentiometer_Bourns_3339P_Vertical_large" (id 2) (at 149.86 69.85 0)
       (effects (font (size 1.27 1.27)) hide)
     )
@@
     (pin "2")
     (pin "3")
+  )
+  (symbol (lib_id "Jumper:Jumper_2_Open") (at 137.16 143.51 0) (unit 1)
+    (in_bom yes) (on_board yes) (fields_autoplaced)
+    (property "Reference" "JP1" (id 0) (at 137.16 140.6962 0))
+    (property "Value" "Jumper_2_Open" (id 1) (at 137.16 140.6961 0)
+      (effects (font (size 1.27 1.27)) hide)
+    )
+    (property "Footprint" "My_Parts:Angled_Jumper_1x02_P2.54mm_large" (id 2) (at 137.16 143.51 0)
+      (effects (font (size 1.27 1.27)) hide)
+    )
+    (property "Datasheet" "~" (id 3) (at 137.16 143.51 0)
+      (effects (font (size 1.27 1.27)) hide)
+    )
+    (pin "1")
+    (pin "2")
   )
   (sheet_instances
@@
       (reference "J1") (unit 1) (value "10-pin_header_LCD_interface") (footprint "My_Headers:10-pin_LCD_header_larger_pads")
     )
-    (path "/00000000-0000-0000-0000-00005e5ec4a7"
-      (reference "J2") (unit 1) (value "Conn_01x02_Male") (footprint "My_Misc:PinHeader_1x02_P2.54mm_Vertical_larger_pads")
+    (path "/885a302b-f7eb-45c8-a6b9-2028e2ac70ed"
+      (reference "JP1") (unit 1) (value "Jumper_2_Open") (footprint "My_Parts:Angled_Jumper_1x02_P2.54mm_large")
     )
     (path "/00000000-0000-0000-0000-00005e3b2793"
@@
     )
     (path "/5939b271-8f38-46ac-b012-8f58b3d290ac"
-      (reference "RV?") (unit 1) (value "R_Potentiometer") (footprint "")
+      (reference "RV1") (unit 1) (value "Contrast") (footprint "My_Misc:Potentiometer_Bourns_3339P_Vertical_large")
     )
     (path "/00000000-0000-0000-0000-00005e3b0f7f"
-      (reference "U1") (unit 1) (value "LCD_HD44780") (footprint "My_Headers:16-pin_LCD_header_larger_pads")
-    )
-  )
+      (reference "U1") (unit 1) (value "LCD_HD44780") (footprint "My_Parts:LCD_HD44780_16x2_w_headers_no outlinelarge")
+    )
+  )
