File: ESPxx Programmer/ESPxx Programmer.kicad_sch (KiCad schematic)
At the start: 7 parts

Commit message: ESPxxProgrammer
Parts:
- added C1, C2: 22u, My_Misc:CP_Radial_D5.0mm_P2.00mm_larger, symbol Device:C_Polarized
- added J1: FTDI Programmer, My_Headers:6-pin FTDI Programmer PinSocket large, symbol My_Headers:6-pin_FTDI_Programmer_socket
- added U3: AMS1117-3.3, Package_TO_SOT_SMD:SOT-223-3_TabPin2, symbol Regulator_Linear:AMS1117-3.3
- added U4: Level shifter BSS138, My_Parts:4-channel_I2C_level_shifter_BSS138_large, symbol My_Parts:4-channel_I2C_level_shifter_BSS138
- JP1: renamed from JP?; value (none) -> Flash; footprint (none) -> My_Parts:Jumper_1x02_P2.54mm_large
- R1, R2: renamed from R?; value (none) -> 10k; footprint (none) -> My_Misc:R_Axial_DIN0207_L6.3mm_D2.5mm_P10.16mm_Horizontal_larger_pads
- SW1: renamed from SW?; value (none) -> Flash; footprint (none) -> My_Misc:SW_PUSH-12mm_large
- SW2: renamed from SW?; value (none) -> Reset; footprint (none) -> My_Misc:SW_PUSH-12mm_large
- U1: renamed from U?; footprint ESP32-CAM -> My_ESP32:ESP32-CAM
- U2: renamed from U?; value (none) -> ESP-01h; footprint (none) -> My_ESP8266:ESP-01_w_pin_socket_large
Connections:
- net +3V3: now also C2.1, U3.2 (VO), U4.6 (LV)
- net +5V: now also C1.1, J1.3 (VCC), U3.3 (VI), U4.12 (HV)
- net GND: now also C1.2, C2.2, J1.1 (GND), U3.1 (GND), U4.1 (GND), U4.7 (GND)
- net RX: now also J1.5 (RX), U4.11 (B1); no longer U2.2 (GPIO1/UOTxD)
- net TX: now also J1.4 (TX), U4.10 (B2); no longer U2.7 (GPIO3/UORxD)
- new net RX-l: U2.2 (GPIO1/UOTxD), U4.5 (A1)
- new net TX-l: U2.7 (GPIO3/UORxD), U4.4 (A2)
