File: 3PinLCDBackpack/3PinLCDBackpack.kicad_pcb (KiCad board)
At the start: 2 copper layers, 54 x 19.7 mm, 8 parts, among them Q1 BC547, U1 74HC595, U2 LCD_HD44780, U3 5-pin_LiquidCrystal595_connec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

Commit message: 3pinlcd
Other:
- board text added: "${TITLE}-${REVISION} Design: Jon Sagebrand github.com/jonsag/miscPCBs"
- board text removed: "3PinLCDBackpack Design: Jon Sagebrand github.com/jonsag/miscPCBs"
Changed lines of the file:
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@@
   )
   (paper "A4")
+  (title_block
+    (title "3PinLCDBackPack")
+    (date "2022-09-09")
+    (rev "0.1")
+  )
   (layers
     (0 "F.Cu" signal)
@@
     (effects (font (size 0.762 0.762) (thickness 0.127)) (justify mirror))
   )
-  (gr_text "3PinLCDBackpack\nDesign: Jon Sagebrand\ngithub.com/jonsag/miscPCBs" (at 174.625 66.04) (layer "B.SilkS")
+  (gr_text "${TITLE}-${REVISION}\nDesign: Jon Sagebrand\ngithub.com/jonsag/miscPCBs" (at 174.625 66.04) (layer "B.SilkS")
     (effects (font (size 0.762 0.762) (thickness 0.127)) (justify left mirror))
   )
