File: Uber I2C LCD Controller Module/KiCad/Uber I2C LCD Controller Module/Uber I2C LCD Controller Module.kicad_pcb (KiCad board)
At the start: 2 copper layers, 38 parts, among them J1 I2C_Interface, Q1 2N7000, Q2 2N7000, Q3 BC237, Q4 BC557B, Q5 BC237, U1 L78L33_TO92, U2 MCP41010, U3 PCF8574N, U4 LCD_HD44780, U5 ATtiny85-20P

Commit message: ...
Parts:
- D1, J1, JP1, JP2, JP3, JP4, JP5, JP6, RV1: moved to B.Cu
- moved J1 108.4 mm to (111.1, 81.8)
- moved R7 86.6 mm to (151.8, 70.5)
- moved D1 83.5 mm to (127.6, 66.7)
- moved C3 82.4 mm to (167.0, 69.8), turned to 180 degrees
- moved R13 79.7 mm to (171.4, 67.3), turned to 90 degrees
- moved R14 77.4 mm to (116.2, 71.8)
- moved U2 76.5 mm to (162.6, 73.7)
- moved C2 73.6 mm to (122.6, 67.9), turned to 90 degrees
- moved RV1 73.0 mm to (176.4, 76.8), turned to 180 degrees
- moved C1 72.9 mm to (109.9, 67.9), turned to 90 degrees
- moved R11 69.4 mm to (156.2, 57.1), turned to -90 degrees
- moved U1 66.3 mm to (115.6, 67.0)
- moved R5 64.9 mm to (135.3, 78.1), turned to 90 degrees
- moved R6 62.7 mm to (139.7, 87.0), turned to 180 degrees
- moved JP1 60.8 mm to (175.9, 81.3), turned to 180 degrees
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Routing:
- net GND: track 0.00 -> 198.3 mm
- net +5V: track 0.00 -> 179.9 mm
- net SDA_H: track 0.00 -> 82.7 mm, vias 0 -> 1
- net Contrast: track 0.00 -> 79.1 mm, vias 0 -> 1
- net SCL_H: track 0.00 -> 69.4 mm, vias 0 -> 1
- net A: track 0.00 -> 46.5 mm
- net RS: track 0.00 -> 43.6 mm, vias 0 -> 1
- net RW: track 0.00 -> 37.0 mm, vias 0 -> 1
- net Net-(Q3-C): track 0.00 -> 35.0 mm
- net Net-(JP3-B): track 0.00 -> 31.7 mm, vias 0 -> 2
- net En: track 0.00 -> 31.7 mm, vias 0 -> 1
- net Net-(JP2-B): track 0.00 -> 28.0 mm
- net SCL: track 0.00 -> 27.6 mm
- net DB5: track 0.00 -> 27.0 mm
- net DB7: track 0.00 -> 26.9 mm
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Other:
- board outline added: 80 x 36.2 mm
