File: RPi IR Receiver/KiCAD/RPi-LibreELEC IR Receiver/RPi-LibreELEC IR Receiver.kicad_sch (KiCad schematic)
At the start: 6 parts, among them J2 Raspberry_Pi_2_3_pin_ordered, Q1 BC547B, U1 TSOP38238

Commit message: RPi IR
Parts:
- J2: footprint (none) -> My_RaspberryPi:RaspberryPi_Hat_2x20_pin_GPIO_larger_pads
- Q1: footprint Package_TO_SOT_THT:TO-92_Inline -> My_Misc:TO-92_Inline_Wide_large
- R1, R2: footprint (none) -> My_Misc:R_Axial_DIN0207_L6.3mm_D2.5mm_P10.16mm_Horizontal_large
Connections:
- net GND: now reaches J2.6 (GND), Q1.3 (E), U1.2 (GND)
- net 3V3: now reaches J2.1 (3V3), R2.1, U1.3 (Vs)
Changed lines of the file:
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@@
+		)
+	)
+	(label "GND"
+		(at 132.08 156.21 0)
+		(effects
+			(font
+				(size 1.27 1.27)
+			)
+			(justify left bottom)
+		)
+	)
+	(label "3V3"
+		(at 132.08 69.85 0)
+		(effects
+			(font
+				(size 1.27 1.27)
+			)
+			(justify left bottom)
 		)
 	)
@@
 			)
 		)
-		(property "Footprint" ""
+		(property "Footprint" "My_Misc:R_Axial_DIN0207_L6.3mm_D2.5mm_P10.16mm_Horizontal_large"
 			(at 110.49 135.128 90)
 			(effects
@@
 			)
 		)
-		(property "Footprint" "Package_TO_SOT_THT:TO-92_Inline"
+		(property "Footprint" "My_Misc:TO-92_Inline_Wide_large"
 			(at 86.36 135.255 0)
 			(effects
@@
 			)
 		)
-		(property "Footprint" ""
+		(property "Footprint" "My_Misc:R_Axial_DIN0207_L6.3mm_D2.5mm_P10.16mm_Horizontal_large"
 			(at 87.122 96.52 90)
 			(effects
@@
 			)
 		)
-		(property "Footprint" ""
+		(property "Footprint" "My_RaspberryPi:RaspberryPi_Hat_2x20_pin_GPIO_larger_pads"
 			(at 160.02 113.03 0)
 			(effects
